Commit message: fix URDF

File: rto_description/urdf/sensors/hokuyo.urdf.xacro (robot description, xacro)
@@ -5,13 +5,4 @@
   <xacro:property name="HOKUYO_RADIUS" value="0.02"/>
   <xacro:property name="HOKUYO_LENGTH" value="0.07"/>
-  <xacro:property name="USE_GPU" value="false"/>
-  <xacro:if value="${USE_GPU}">
-    <xacro:property name="LASER_TYPE" value="gpu_ray"/>
-    <xacro:property name="FILENAME" value="libgazebo_ros_gpu_laser.so"/>
-  </xacro:if>
-  <xacro:unless value="${USE_GPU}">
-    <xacro:property name="LASER_TYPE" value="ray"/>
-    <xacro:property name="FILENAME" value="libgazebo_ros_laser.so"/>
-  </xacro:unless>
   <xacro:macro name="hokuyo" params="parent name *origin">
     <joint name="${name}_joint" type="fixed">
@@ -47,5 +38,5 @@
   <xacro:macro name="hokuyo_gazebo" params="name ros_topic update_rate min_angle max_angle">
     <gazebo reference="${name}_link">
-      <sensor name="${name}" type="${LASER_TYPE}">
+      <sensor name="${name}" type="gpu_ray">
         <!--always_on>true</always_on-->
         <update_rate>40</update_rate>
@@ -72,5 +63,5 @@
           </noise>
         </ray>
-        <plugin name="gazebo_ros_${name}_controller" filename="${FILENAME}">
+        <plugin name="gazebo_ros_${name}_controller" filename="libgazebo_ros_gpu_laser.so">
           <topicName>${ros_topic}</topicName>
           <frameName>${name}_link</frameName>
